Commit message: Decreased the tactip tip coillision scale for getting larger contact depth images

File: urdf/robots/tactile_sim_assets/embodiment_assets/combined_urdfs/right_angle_tactip.urdf (robot description, URDF)
Before this commit: robot universal_robot, 14 links, 13 joints
Links:
- link tactip_tip_link: geometry collision mesh filename=../sensor_assets/right_angle_tactip/../standard_tactip/tip/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 scale=1.00000 0.9 1.0; visual mesh filename=../sensor_assets/right_angle_tactip/../standard_tactip/tip/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 scale=1.00000 1.00000 1.00000
