Commit message: added leap hand with tactile sensors

File: urdf/robots/tactile_sim_assets/embodiment_assets/combined_urdfs/ur5_leap_hand_tactip_data_collect.urdf (robot description, URDF)
Before this commit: robot universal_robot, 15 links, 14 joints
Links:
- removed link elastomer_tip
- removed link fake_tcp_link_for_tactile_image
- added link adaptor_link, mass 0.18790; visual mesh filename=package://tactile_sim_assets/sensor_assets/leap_hand_tactip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 scale=0.001 0.00100 0.00100
- link tactip_body_link: geometry visual mesh filename=package://tactile_sim_assets/sensor_assets/leap_hand_tactip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 scale=1.00000 1.00000 1.00000
- link tactip_tip_link: geometry visual mesh filename=package://tactile_sim_assets/sensor_assets/leap_hand_tactip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 scale=0.00106 0.001044 0.001044
Joints:
- removed joint dummy_camera_joint
- removed joint fake_tcp_joint
- added joint adaptor_joint: type fixed, parent ee_link, child adaptor_link, origin xyz=-0.015 0.02 -0.007 rpy=1.57 0 -1.57, axis 0.00000 0.00000 0.00000
- joint camera_joint: origin xyz=0.00000 0.00000 0.06500 rpy=0 0.000 0.000 -> xyz=0.0 0.005 -0.0255 rpy=0.0 0.0 -1.5708; parent tactip_body_link -> tactip_tip_link
- joint joint_dummy1: origin xyz=0.00000 0.00000 0.00000 rpy=-3.14159 0.00000 3.14159 -> xyz=0.00000 0.0138000 -0.06750000 rpy=1.57 3.14 0
- joint tactip_tip_to_body: origin xyz=0.00000 0.00000 0.06500 rpy=1.57000 -0.00000 0.00000 -> xyz=0 0 0 rpy=1.5707963267949 0 3.14159265358979
- joint tcp_joint: origin xyz=0.00000 0.00000 0.06500 rpy=0 0.000 0.000 -> xyz=0.0 0.005 -0.0205 rpy=0.0 0.0 -1.5708; parent tactip_body_link -> tactip_tip_link
